File: kibot-test-cicd.kicad_sch (KiCad schematic)
At the start: 0 parts

Commit message: [added] completed initial sch design, move from draft to preliminary
Other:
- note added: "This board is meant to validate the magnetic encoder MT6701"
- note removed: "Comment"
- title: (none) -> Cover Page
