File: kibot-test-cicd.kicad_pcb (KiCad board)
At the start: 6 copper layers, 0 parts

Commit message: [PCB] added basic layout
Parts:
- added C1: 0.1uF, Capacitor_SMD:C_0603_1608Metric, F.Cu at (143.8, 88.9)
- added D1: ESD9B3.3ST5G, Diode_SMD:D_SOD-923, F.Cu at (160.5, 90.9)
- added D2: LED, LED_SMD:LED_0603_1608Metric, F.Cu at (144.8, 101.6)
- added H1: M3, MountingHole:MountingHole_3.2mm_M3, F.Cu at (137.1, 78.4)
- added H2: M3, MountingHole:MountingHole_3.2mm_M3, F.Cu at (158.8, 102.9)
- added H3: M3, MountingHole:MountingHole_3.2mm_M3, F.Cu at (158.8, 78.5)
- added H4: M3, MountingHole:MountingHole_3.2mm_M3, F.Cu at (137.1, 102.3)
- added J1: Conn_02x04_Counter_Clockwise, Connector_PinHeader_2.54mm:PinHeader_2x04_P2.54mm_Vertical, F.Cu at (133.4, 94.0)
- added J2: Conn_01x05_Pin, Connector_JST:JST_SH_BM05B-SRSS-TB_1x05-1MP_P1.00mm_Vertical, F.Cu at (163.8, 90.2)
- added JP1: SolderJumper_2_Bridged, Jumper:SolderJumper-2_P1.3mm_Bridged_RoundedPad1.0x1.5mm, F.Cu at (146.1, 105.4)
- added R1: 5k, Resistor_SMD:R_0402_1005Metric, F.Cu at (147.8, 102.9)
- added U1: MT6701CT, Package_SO:SO-8_3.9x4.9mm_P1.27mm, B.Cu at (148.5, 90.0)
Other:
- board outline added: 47 x 47 mm
